Commit message: dummy link added

File: kr_robot_description/kr810/urdf/kr810_description.urdf.xacro (robot description, xacro)
@@ -57,4 +57,5 @@
       </collision>
   </xacro:macro>
+  <link name="world"/>
   <link name="base">
     <xacro:property name="base_outer_radius" value="${ 80 * scale}" />
@@ -317,4 +318,8 @@
   </link>
   <!-- joints -->
+  <joint name="dummy" type="fixed">
+    <parent link="world"/>
+    <child link="base"/>
+  </joint>
   <joint name="joint_1" type="continuous">
     <parent link="base"/>

File: kr_robot_driver/description/urdf/kr810.urdf.xacro (robot description, xacro)
@@ -3,6 +3,4 @@
   <!-- Import kr810 macro -->
   <xacro:include filename="$(find kr_robot_description)/kr810/urdf/kr810_description.urdf.xacro"/>
-  <!-- create link fixed to the "world" -->
-  <!-- <link name="world"/> -->
   <xacro:kr810_description/>
   <!-- Import r6bot ros2_control description -->
